File: xbee thing/Grove  - XBee Carrier v1.0.brd (EAGLE design)
At the start: 46.5 x 50.9 mm, 38 parts, among them J1 SULLINS_NPPN101BFCN-RCSULLINS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, J2 HEADER-10P_STANDARD, J3 HEADER-10P_STANDARD, J4 SULLINS_NPPN101BFCN-RCSULLINS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, J5 105450-0101, Q1 Si2305DS, Q2 Si2305DS, Q3 Si2305DS, U2 RT9167A_33PB, U3 CN3083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

Commit message: yote
Parts:
- added J6: (no value), SparkFun-Connectors:USB-C-16P
- added R12, R13, R2, R6: 5.1K, discrete:0603
- J5: value 105450-0101 -> (none); device 105450-0101:MOLEX_105450-0101 -> SparkFun-Connectors:USB-C-16P
- moved J5 48.6 mm to (5.71, 0.00), flipped to the top, turned to 0 degrees
Connections:
- removed net A1: J1.8, J3.8, J5.A7, J5.B7, X3.2
- removed net AREF: J1.7, J3.7, J5.A6, J5.B6, X3.3
- new net D_2+: J1.7, J3.7, J6.A6, J6.B6, X3.3
- new net D_2-: J1.8, J3.8, J6.A7, J6.B7, X3.2
- new net N$13: J6.B5, R6.2
- new net N$14: J5.B5, R13.2
- new net N$3: U4.17
- new net N$4: J6.A5, R2.2
- new net N$5: J5.A5, R12.2
- net D+: now also J5.A6, J5.B6
- net D-: now also J5.A7, J5.B7
- net GND: now also J5.GND, J5.GND2, J6.GND, J6.GND2, R12.1, R13.1, R2.1, R6.1; no longer J5.A1, J5.A12, J5.B1, J5.B12
- net N$10: no longer U4.17
- net USB_5V: now also J5.VBUS1, J5.VBUS2, J6.VBUS1, J6.VBUS2; no longer J5.A4, J5.A9, J5.B4, J5.B9
Routing:
- net D_2-: track 0.00 -> 47.8 mm, vias 0 -> 1
- net A1: track 47.8 -> 0.00 mm, vias 1 -> 0
- net D_2+: track 0.00 -> 44.2 mm, vias 0 -> 1
- net AREF: track 44.2 -> 0.00 mm, vias 1 -> 0
- net USB_5V: track 85.0 -> 82.2 mm
- net N$10: track 3.24 -> 2.38 mm

Commit message: screm usbc
Parts:
- removed X3, X4: MINI-USB-UX60A-MB-5ST, con-hirose:UX60A-MB-5ST
- added U1: TUSB2046BVF, TUSB2046BVF:QFP80P900X900X145-32N
- R12, R13, R2, R6: value 5.1K -> (none)
- moved R13 76.2 mm to (31.1, 42.7), flipped to the bottom, turned to 90 degrees
- moved R12 72.5 mm to (29.2, 42.7), flipped to the bottom, turned to 90 degrees
- moved R6 68.9 mm to (27.3, 42.7), flipped to the bottom, turned to 90 degrees
- moved R2 65.2 mm to (25.4, 42.7), flipped to the bottom, turned to 90 degrees
- moved J6 56.5 mm to (20.3, 45.7), flipped to the bottom, turned to 180 degrees
- moved J5 54.6 mm to (35.6, 45.7), flipped to the bottom, turned to 180 degrees
Connections:
- removed net N$10: U4.19
- removed net N$3: U4.17
- new net N$17: J2.1, J4.10
- new net VCC: U1.3
- new net VCC_2: U1.25
- net D+: no longer X4.3
- net D-: no longer X4.2
- net D_2+: no longer X3.3
- net D_2-: no longer X3.2
- net GND: now also U1.28, U1.31, U1.7; no longer J2.1, J4.10, X3.5, X4.5
- net USB_5V: no longer X3.1, X4.1
- net VCC_3V3: now also U1.8
Routing:
- net GND: track 28.9 -> 65.6 mm
- net N$4: track 0.00 -> 7.61 mm
- net N$14: track 0.00 -> 7.45 mm
- net D+: track 34.0 -> 41.5 mm, vias 0 -> 2
- net N$13: track 0.00 -> 6.38 mm
- net N$5: track 0.00 -> 6.29 mm
- net D-: track 34.4 -> 39.5 mm, vias 0 -> 2
- net USB_5V: track 82.2 -> 78.6 mm
- net D_2-: track 47.8 -> 45.4 mm
- net N$10: track 2.38 -> 0.00 mm
- net D_2+: track 44.2 -> 45.2 mm

Commit message: haha nou
Parts:
- removed J5, J6: (no value), SparkFun-Connectors:USB-C-16P
- removed R12, R13, R2, R6: (no value), discrete:0603
- added C10: 15v-10uF, discrete:AVX-A
- added C9: 15v-27pF, discrete:AVX-A
- added J7: (no value), SparkFun-Connectors:USB-C-16P
- added Q4: FQ7050B-6.000, FQ7050B-6.000:FQ7050B
- added R14, R15: (no value), discrete:0603
Connections:
- removed net N$13: J6.B5, R6.2
- removed net N$14: J5.B5, R13.2
- removed net N$4: J6.A5, R2.2
- removed net N$5: J5.A5, R12.2
- removed net VCC: U1.3
- new net N$10: J7.B5, R15.2
- new net N$3: J7.A5, R14.2
- new net ROOTD+: J7.A6, J7.B6, U1.1
- new net ROOTD-: J7.A7, J7.B7, U1.2
- new net XTAL1: C9.+, Q4.1, U1.30
- new net XTAL2: C10.+, Q4.4, U1.29
- net D+: now also U1.12; no longer J5.A6, J5.B6
- net D-: now also U1.11; no longer J5.A7, J5.B7
- net D_2+: now also U1.16; no longer J6.A6, J6.B6
- net D_2-: now also U1.15; no longer J6.A7, J6.B7
- net GND: now also C10.-, C9.-, J7.GND, J7.GND2, R14.1, R15.1, U1.27, U1.8; no longer J5.GND, J5.GND2, J6.GND, J6.GND2, R12.1, R13.1, R2.1, R6.1
- net USB_5V: now also J7.VBUS1, J7.VBUS2; no longer J5.VBUS1, J5.VBUS2, J6.VBUS1, J6.VBUS2
- net VCC_3V3: now also U1.3; no longer U1.8
Routing:
- net GND: track 65.6 -> 28.9 mm
- net USB_5V: track 78.6 -> 62.5 mm
- net D+: track 41.5 -> 30.1 mm, vias 2 -> 0
- net D_2-: track 45.4 -> 34.3 mm, vias 1 -> 0
- net D-: track 39.5 -> 29.3 mm, vias 2 -> 0
- net N$4: track 7.61 -> 0.00 mm
- net N$14: track 7.45 -> 0.00 mm
- net D_2+: track 45.2 -> 37.8 mm, vias 1 -> 0
- net N$13: track 6.38 -> 0.00 mm
- net N$5: track 6.29 -> 0.00 mm

Commit message: maybe impl'd hub, delet battery stuff
Parts:
- removed C5: 1.0uF, SparkFun-Capacitors:0805
- removed C8: 10V-22uF, discrete:AVX-B
- removed CH: RED, discrete:D0603
- removed D1, D2, D3: SS14, discrete:D2010
- removed OK: Green, discrete:D0603
- removed Q1: Si2305DS, discrete:SOT23
- removed R10: 10K, discrete:0603
- removed R4: 1k, discrete:0603
- removed R8: 3.9K, discrete:0603
- removed U3: CN3083, IC:SOP8
- added C6: 15v-1uF, discrete:AVX-A
- added R12, R13, R2: 15k, discrete:0603
- added R6: 10k, discrete:0603
- R14, R15: value (none) -> 5.1k
- flipped C10 to the bottom
- flipped C9 to the bottom
- flipped J7 to the bottom
- flipped Q4 to the bottom
- flipped R14 to the bottom
- flipped R15 to the bottom
- flipped U1 to the bottom
Connections:
- removed net HEAT: U3.HEAT
- removed net N$11: D3.-, Q1.2
- removed net N$2: R8.2, U3.2
- removed net N$7: CH.-, U3.7
- removed net N$8: OK.-, U3.6
- removed net N$9: CH.+, OK.+, R4.1
- removed net VBET: C5.2, D3.+, U3.5, U3.8
- removed net VCC_2: U1.25
- removed net VIN: C8.+, D2.-, R4.2, U3.4
- new net HUB_RESET: C6.+, R2.2, U1.4
- new net N$5: R6.1, U1.10, U1.14, U1.18, U1.22
- net D+: now also R12.2
- net D_2+: now also R13.2
- net GND: now also C6.-, R12.1, R13.1; no longer C5.1, C8.-, R10.1, R8.1, U3.1, U3.3
- net USB_5V: no longer D1.+, D2.+, Q1.1, R10.2
- net VBET_OUT: no longer D1.-, Q1.3
- net VCC_3V3: now also R2.1, R6.2, U1.25, U1.26, U1.6
Routing:
- net USB_5V: track 62.5 -> 31.2 mm, vias 4 -> 2
- net N$8: track 31.1 -> 0.00 mm, vias 2 -> 0
- net N$7: track 30.8 -> 0.00 mm, vias 2 -> 0
- net VIN: track 25.8 -> 0.00 mm, vias 2 -> 0
- net VBET_OUT: track 51.0 -> 27.0 mm, vias 2 -> 0
- net VBET: track 21.1 -> 0.00 mm
- net GND: track 28.9 -> 10.0 mm, vias 9 -> 8
- net D_2+: track 37.8 -> 29.7 mm
- net N$11: track 6.63 -> 0.00 mm
- net N$2: track 5.11 -> 0.00 mm
- net N$9: track 3.33 -> 0.00 mm
- net D_2-: track 34.3 -> 35.0 mm

Commit message: Maybe fixed it
Parts:
- removed Q2, Q3: Si2305DS, discrete:SOT23
- added 5V, GND, PDM, PDP: (no value), wirepad:2,15/1,0
- moved R13 85.5 mm to (26.7, 22.2), flipped to the bottom
- moved R12 84.5 mm to (26.7, 24.1), flipped to the bottom
- moved R6 71.9 mm to (25.1, 11.8), flipped to the bottom
- moved R14 69.2 mm to (34.9, 41.9), turned to 90 degrees
- moved R15 68.0 mm to (36.8, 41.9), turned to 90 degrees
- moved J7 63.3 mm to (35.6, 45.7), turned to 180 degrees
- moved C6 55.2 mm to (14.6, 9.53), turned to 270 degrees
- moved R2 53.9 mm to (16.5, 9.53), turned to 90 degrees
- moved C10 45.4 mm to (14.6, 4.45), turned to 270 degrees
- moved C9 43.7 mm to (16.5, 4.45), turned to 270 degrees
- moved Q4 40.0 mm to (20.3, 6.35), turned to 270 degrees
- moved U1 30.5 mm to (21.6, 17.8), turned to 180 degrees
Connections:
- net N$10 renamed USBC_CC2
- net N$3 renamed USBC_CC1
- net N$5 renamed USB_OVRCUR
- removed net VBET_OUT: C1.1, U2.1, U2.3
- removed net VCC_OUT1: Q3.3
- removed net VCC_OUT2: Q2.3
- net GND: now also GND.1, J7.SHLD1, J7.SHLD2, J7.SHLD3, J7.SHLD4, J7.SHLD5, J7.SHLD6, J7.SHLD7, J7.SHLD8
- net PWR_CTR1: no longer Q3.1
- net PWR_CTR2: no longer Q2.1
- net ROOTD+: now also PDP.1
- net ROOTD-: now also PDM.1
- net USB_5V: now also 5V.1, C1.1, U2.1, U2.3
- net VCC_3V3: no longer Q2.2, Q3.2
Routing:
- net ROOTD+: track 0.00 -> 65.4 mm, vias 0 -> 2
- net ROOTD-: track 0.00 -> 60.8 mm, vias 0 -> 4
- net USB_5V: track 31.2 -> 82.7 mm
- net VBET_OUT: track 27.0 -> 0.00 mm
- net D-: track 29.3 -> 7.07 mm
- net USB_OVRCUR: track 0.00 -> 21.1 mm
- net D+: track 30.1 -> 9.56 mm
- net HUB_RESET: track 0.00 -> 20.2 mm, vias 0 -> 2
- net DTR: track 60.8 -> 43.4 mm
- net D_2-: track 35.0 -> 20.5 mm, vias 0 -> 1
- net XTAL2: track 0.00 -> 14.0 mm
- net D4: track 15.3 -> 5.46 mm
- net PWR_CTR1: track 13.5 -> 3.80 mm
- net XTAL1: track 0.00 -> 9.46 mm
- net D_2+: track 29.7 -> 21.8 mm, vias 0 -> 1
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- removed copper zone on layer 1, net HEAT
- removed copper zone on layer 16, net HEAT
Other:
- outline, holes or cut-outs redrawn

Commit message: haha yes
Parts:
- added R10: 1.5k, discrete:0603
- added R4, R8: 15k, discrete:0603
- added USB2M, USB2P, XBM, XBP: (no value), wirepad:2,15/1,0
- flipped J1 to the bottom
- flipped J4 to the bottom
Connections:
- net D+: now also XBP.1
- net D-: now also R4.2, XBM.1
- net D_2+: now also USB2P.1
- net D_2-: now also R8.2, USB2M.1
- net GND: now also R4.1, R8.1
- net ROOTD+: now also R10.2
- net VCC_3V3: now also R10.1
Routing:
- net D-: track 7.07 -> 48.3 mm
- net D+: track 9.56 -> 43.0 mm
- net D_2-: track 20.5 -> 33.8 mm, vias 1 -> 5
- net D_2+: track 21.8 -> 27.3 mm, vias 1 -> 3
- net VCC_3V3: track 110.9 -> 113.1 mm
- net ROOTD+: track 65.4 -> 67.5 mm
- net ASSOC: vias 0 -> 2
- net TX: vias 2 -> 1
- net SDA: vias 0 -> 1
- net RESET: vias 0 -> 1
- net PWR_CTR1: vias 0 -> 1
- net N$17: vias 0 -> 1
- net DTR: vias 1 -> 2
- net D9: vias 0 -> 1
- net D8: vias 0 -> 1
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
Commit message: plz dont break
Routing:
- net USB_5V: track 82.7 -> 84.5 mm
Changed lines of the file:
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@@
 <drawing>
 <settings>
-<setting alwaysvectorfont="yes"/>
+<setting alwaysvectorfont="no"/>
 <setting keepoldvectorfont="yes"/>
 <setting verticaltext="up"/>
@@
 <wire x1="41.0617" y1="38.54878125" x2="38.01" y2="41.60048125" width="0.6096" layer="16"/>
 <wire x1="38.01" y1="41.60048125" x2="38.01" y2="45.566" width="0.6096" layer="16"/>
-<wire x1="30.3582" y1="27.8182" x2="31.115" y2="28.575" width="0.6096" layer="16"/>
-<via x="31.115" y="28.575" extent="1-16" drill="0.35"/>
-<wire x1="31.115" y1="28.575" x2="37.2094" y2="34.6694" width="0.6096" layer="16"/>
+<wire x1="30.3582" y1="27.8182" x2="31.4325" y2="28.8925" width="0.6096" layer="16"/>
+<wire x1="31.4325" y1="28.8925" x2="37.2094" y2="34.6694" width="0.6096" layer="16"/>
 <wire x1="37.2094" y1="34.6694" x2="37.35471875" y2="34.6694" width="0.6096" layer="16"/>
 <wire x1="37.35471875" y1="34.6694" x2="37.55791875" y2="34.8726" width="0.6096" layer="16"/>
-<wire x1="31.115" y1="28.575" x2="28.194" y2="25.654" width="0.6096" layer="1"/>
-<wire x1="28.194" y1="25.654" x2="22.987" y2="25.654" width="0.6096" layer="1"/>
 <contactref element="5V" pad="1"/>
 <wire x1="33.4522" y1="47.489" x2="33.4522" y2="46.841" width="0.4064" layer="16"/>
@@
 <wire x1="32.0462" y1="48.895" x2="33.4522" y2="47.489" width="0.4064" layer="16"/>
 <wire x1="27.305" y1="48.895" x2="32.0462" y2="48.895" width="0.4064" layer="16"/>
+<wire x1="31.4325" y1="28.8925" x2="31.4325" y2="27.6225" width="0.6096" layer="16"/>
+<wire x1="31.4325" y1="27.6225" x2="31.75" y2="27.305" width="0.6096" layer="16"/>
+<via x="31.75" y="27.305" extent="1-16" drill="0.35"/>
+<wire x1="31.75" y1="27.305" x2="30.099" y2="25.654" width="0.8128" layer="1"/>
+<wire x1="30.099" y1="25.654" x2="22.987" y2="25.654" width="0.8128" layer="1"/>
 </signal>
 <signal name="D-">
@@
 <via x="16.51" y="43.18" extent="1-16" drill="0.35"/>
 </signal>
+<signal name="N$3">
+<via x="26.67" y="27.94" extent="1-16" drill="0.35"/>
+</signal>
 </signals>

Commit message: Maybe at least a little fix the things it's complaining about?
Routing:
- net DTR: track 43.4 -> 44.8 mm, vias 2 -> 1
- net D_2+: track 27.3 -> 28.4 mm, vias 3 -> 2
- net N$17: track 4.11 -> 3.89 mm, vias 1 -> 0
- net D5: track 8.79 -> 8.59 mm, vias 1 -> 0
- net PWR_CTR1: track 3.80 -> 3.75 mm, vias 1 -> 0
- net D_2-: vias 5 -> 4
- net D8: vias 1 -> 0
- net D7: track 4.56 -> 4.57 mm, vias 1 -> 0
- net RESET: track 5.23 -> 5.24 mm, vias 1 -> 0
- net D9: vias 1 -> 0
- net D4: vias 1 -> 0
- net SDA: track 6.40 -> 6.41 mm, vias 1 -> 0
- net ASSOC: vias 2 -> 0
