File: xbee thing/Grove  - XBee Carrier v1.0.sch (EAGLE design)
At the start: 38 parts, among them J1 SULLINS_NPPN101BFCN-RCSULLINS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, J2 HEADER-10P_STANDARD, J3 HEADER-10P_STANDARD, J4 SULLINS_NPPN101BFCN-RCSULLINS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, J5 105450-0101, Q1 Si2305DS, Q2 Si2305DS, Q3 Si2305DS, U2 RT9167A_33PB, U3 CN3083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

Commit message: yote
Parts:
- added J6: (no value), SparkFun-Connectors:USB_C2-LAYER
- added R12, R13, R2, R6: 5.1K, discrete:R-0603
- J5: value 105450-0101 -> (none); device 105450-0101:105450-0101 -> SparkFun-Connectors:USB_C2-LAYER
Connections:
- removed net A1: J1.8, J3.8, J5.D1-, J5.D2-, X3.2
- removed net AREF: J1.7, J3.7, J5.D1+, J5.D2+, X3.3
- new net D_2+: J1.7, J3.7, J6.D+, X3.3
- new net D_2-: J1.8, J3.8, J6.D-, X3.2
- new net N$13: J6.CC2, R6.2
- new net N$14: J5.CC2, R13.2
- new net N$3: U4.3V3OUT
- new net N$4: J6.CC1, R2.2
- new net N$5: J5.CC1, R12.2
- net D+: now also J5.D+
- net D-: now also J5.D-
- net GND: now also J5.GND, J6.GND, R12.1, R13.1, R2.1, R6.1; no longer J5.GND1, J5.GND2, J5.GND3, J5.GND4
- net N$10: no longer U4.3V3OUT
- net USB_5V: now also J5.VBUS, J6.VBUS; no longer J5.VBUS1, J5.VBUS2, J5.VBUS3, J5.VBUS4

Commit message: screm usbc
Parts:
- removed X3, X4: MINI-USB-UX60A-MB-5ST, con-hirose:MINI-USB-UX60A-MB-5ST
- added U1: TUSB2046BVF, TUSB2046BVF:TUSB2046BVF
- R12, R13, R2, R6: value 5.1K -> (none)
Connections:
- removed net N$10: U4.!RESET
- removed net N$3: U4.3V3OUT
- new net N$17: J2.1, J4.10
- net D+: no longer X4.3
- net D-: no longer X4.2
- net D_2+: no longer X3.3
- net D_2-: no longer X3.2
- net GND: now also U1.GND, U1.GND_2, U1.TSTMODE; no longer J2.1, J4.10, X3.5, X4.5
- net USB_5V: no longer X3.1, X4.1
- net VCC_3V3: now also U1.BUSPWR

Commit message: haha nou
Parts:
- removed J5, J6: (no value), SparkFun-Connectors:USB_C2-LAYER
- removed R12, R13, R2, R6: (no value), discrete:R-0603
- added C10: 15v-10uF, discrete:CAP_AVX_A
- added C9: 15v-27pF, discrete:CAP_AVX_A
- added J7: (no value), SparkFun-Connectors:USB_C2-LAYER
- added Q4: FQ7050B-6.000, FQ7050B-6.000:FQ7050B-6.000
- added R14, R15: (no value), discrete:R-0603
Connections:
- removed net N$13: J6.CC2, R6.2
- removed net N$14: J5.CC2, R13.2
- removed net N$4: J6.CC1, R2.2
- removed net N$5: J5.CC1, R12.2
- new net N$10: J7.CC2, R15.2
- new net N$3: J7.CC1, R14.2
- new net ROOTD+: J7.D+, U1.DP0
- new net ROOTD-: J7.D-, U1.DM0
- new net XTAL1: C9.+, Q4.1, U1.XTAL1
- new net XTAL2: C10.+, Q4.2, U1.XTAL2
- net D+: now also U1.DP1; no longer J5.D+
- net D-: now also U1.DM1; no longer J5.D-
- net D_2+: now also U1.DP2; no longer J6.D+
- net D_2-: now also U1.DM2; no longer J6.D-
- net GND: now also C10.-, C9.-, J7.GND, R14.1, R15.1, U1.BUSPWR, U1.TSTPLL/48MCLK; no longer J5.GND, J6.GND, R12.1, R13.1, R2.1, R6.1
- net USB_5V: now also J7.VBUS; no longer J5.VBUS, J6.VBUS
- net VCC_3V3: now also U1.VCC; no longer U1.BUSPWR

Commit message: maybe impl'd hub, delet battery stuff
Parts:
- removed C5: 1.0uF, SparkFun-Capacitors:1.0UF-0805-25V-10%
- removed C8: 10V-22uF, discrete:CAP_AVX_B
- removed CH: RED, discrete:LED-0603
- removed D1, D2, D3: SS14, discrete:D-2010
- removed OK: Green, discrete:LED-0603
- removed Q1: Si2305DS, discrete:010-P-MOSFETSOT23
- removed R10: 10K, discrete:R-0603
- removed R4: 1k, discrete:R-0603
- removed R8: 3.9K, discrete:R-0603
- removed U3: CN3083, IC:CN3083
- added C6: 15v-1uF, discrete:CAP_AVX_A
- added R12, R13, R2: 15k, discrete:R-0603
- added R6: 10k, discrete:R-0603
- R14, R15: value (none) -> 5.1k
Connections:
- removed net HEAT: U3.HEAT
- removed net N$11: D3.-, Q1.S
- removed net N$2: R8.2, U3.ISET
- removed net N$7: CH.-, U3.CH
- removed net N$8: OK.-, U3.OK
- removed net N$9: CH.+, OK.+, R4.1
- removed net VBET: C5.2, D3.+, U3.BAT, U3.FB
- removed net VIN: C8.+, D2.-, R4.2, U3.VIN
- new net HUB_RESET: C6.+, R2.2, U1.~RESET
- new net N$5: R6.1, U1.~OVRCUR1, U1.~OVRCUR2, U1.~OVRCUR3, U1.~OVRCUR4
- net D+: now also R12.2
- net D_2+: now also R13.2
- net GND: now also C6.-, R12.1, R13.1; no longer C5.1, C8.-, R10.1, R8.1, U3.GND, U3.TEMP
- net USB_5V: no longer D1.+, D2.+, Q1.G, R10.2
- net VBET_OUT: no longer D1.-, Q1.D
- net VCC_3V3: now also R2.1, R6.2, U1.EEDATA/GANGED, U1.VCC_2, U1.~EXTMEM
Other:
- note added: "RC for usb hub reset"
- moved on the sheet: R14, R15

Commit message: Maybe fixed it
Parts:
- removed Q2, Q3: Si2305DS, discrete:010-P-MOSFETSOT23
- added 5V, GND, PDM, PDP: (no value), wirepad:2,15/1,0
Connections:
- net N$10 renamed USBC_CC2
- net N$3 renamed USBC_CC1
- net N$5 renamed USB_OVRCUR
- removed net VBET_OUT: C1.1, U2.EN, U2.VIN
- removed net VCC_OUT1: Q3.D
- removed net VCC_OUT2: Q2.D
- net GND: now also GND.P, J7.SHLD
- net PWR_CTR1: no longer Q3.G
- net PWR_CTR2: no longer Q2.G
- net ROOTD+: now also PDP.P
- net ROOTD-: now also PDM.P
- net USB_5V: now also 5V.P, C1.1, U2.EN, U2.VIN
- net VCC_3V3: no longer Q2.S, Q3.S
Changed lines of the file:
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@@
 <parts>
 <part name="FRAME1" library="frames" library_urn="urn:adsk.eagle:library:229" deviceset="A4L-LOC" device=""/>
-<part name="Q3" library="discrete" library_urn="urn:adsk.eagle:library:211" deviceset="010-P-MOSFET*" device="SOT23" value="Si2305DS"/>
 <part name="PWR" library="discrete" library_urn="urn:adsk.eagle:library:211" deviceset="LED*" device="-0805" value="red"/>
 <part name="R5" library="discrete" library_urn="urn:adsk.eagle:library:211" deviceset="R*" device="-0603" value="1K"/>
@@
 <part name="ASSOC" library="discrete" library_urn="urn:adsk.eagle:library:211" deviceset="LED*" device="-0603" value="Green"/>
 <part name="R11" library="discrete" library_urn="urn:adsk.eagle:library:211" deviceset="R*" device="-0603" value="1K"/>
-<part name="Q2" library="discrete" library_urn="urn:adsk.eagle:library:211" deviceset="010-P-MOSFET*" device="SOT23" value="Si2305DS"/>
 <part name="J2" library="Connector" deviceset="HEADER-10P" device="_STANDARD"/>
 <part name="J3" library="Connector" deviceset="HEADER-10P" device="_STANDARD"/>
@@
 <part name="R12" library="discrete" library_urn="urn:adsk.eagle:library:211" deviceset="R*" device="-0603" value="15k"/>
 <part name="R13" library="discrete" library_urn="urn:adsk.eagle:library:211" deviceset="R*" device="-0603" value="15k"/>
+<part name="5V" library="wirepad" library_urn="urn:adsk.eagle:library:412" deviceset="2,15/1,0" device="" package3d_urn="urn:adsk.eagle:package:30831/1"/>
+<part name="PDM" library="wirepad" library_urn="urn:adsk.eagle:library:412" deviceset="2,15/1,0" device="" package3d_urn="urn:adsk.eagle:package:30831/1"/>
+<part name="PDP" library="wirepad" library_urn="urn:adsk.eagle:library:412" deviceset="2,15/1,0" device="" package3d_urn="urn:adsk.eagle:package:30831/1"/>
+<part name="GND" library="wirepad" library_urn="urn:adsk.eagle:library:412" deviceset="2,15/1,0" device="" package3d_urn="urn:adsk.eagle:package:30831/1"/>
 </parts>
 <sheets>
@@
 <attribute name="SHEET" x="229.235" y="3.81" size="2.54" layer="94" font="vector"/>
 </instance>
-<instance part="Q3" gate="MOS" x="147.32" y="82.55" smashed="yes" rot="R270">
-<attribute name="NAME" x="148.59" y="85.725" size="1.778" layer="95" ratio="10"/>
-<attribute name="VALUE" x="142.24" y="78.105" size="1.778" layer="96" ratio="10"/>
-</instance>
 <instance part="PWR" gate="LED" x="151.13" y="154.94" smashed="yes">
 <attribute name="NAME" x="153.67" y="155.575" size="1.778" layer="95"/>
@@
 <attribute name="VALUE" x="168.275" y="146.05" size="1.778" layer="96" ratio="10" rot="R180"/>
 </instance>
-<instance part="Q2" gate="MOS" x="184.15" y="81.28" smashed="yes" rot="R270">
-<attribute name="NAME" x="184.785" y="84.455" size="1.778" layer="95" ratio="10"/>
-<attribute name="VALUE" x="180.34" y="76.835" size="1.778" layer="96" ratio="10"/>
-</instance>
 <instance part="J2" gate="J" x="138.43" y="118.11" smashed="yes" rot="R180">
 <attribute name="NAME" x="139.7" y="105.41" size="1.778" layer="95" rot="R180"/>
@@
 </instance>
 <instance part="U1" gate="A" x="129.54" y="38.1" smashed="yes">
-<attribute name="NAME" x="126.588790625" y="86.054" size="2.08463125" layer="95" ratio="10" rot="SR0"/>
 <attribute name="VALUE" x="125.42046875" y="1.9143" size="2.085190625" layer="96" ratio="10" rot="SR0"/>
 </instance>
@@
 <attribute name="NAME" x="181.356" y="33.782" size="1.778" layer="95" ratio="10" rot="R180"/>
 <attribute name="VALUE" x="180.721" y="29.972" size="1.778" layer="96" ratio="10" rot="R180"/>
+</instance>
+<instance part="5V" gate="1" x="215.9" y="71.12" smashed="yes">
+<attribute name="NAME" x="209.677" y="70.4342" size="1.778" layer="95"/>
+<attribute name="VALUE" x="214.757" y="67.818" size="1.778" layer="96"/>
+</instance>
+<instance part="PDM" gate="1" x="215.9" y="68.58" smashed="yes">
+<attribute name="NAME" x="207.137" y="67.8942" size="1.778" layer="95"/>
+<attribute name="VALUE" x="214.757" y="65.278" size="1.778" layer="96"/>
+</instance>
+<instance part="PDP" gate="1" x="215.9" y="66.04" smashed="yes">
+<attribute name="NAME" x="207.137" y="65.3542" size="1.778" layer="95"/>
+<attribute name="VALUE" x="214.757" y="62.738" size="1.778" layer="96"/>
+</instance>
+<instance part="GND" gate="1" x="215.9" y="63.5" smashed="yes">
+<attribute name="NAME" x="207.137" y="62.8142" size="1.778" layer="95"/>
+<attribute name="VALUE" x="214.757" y="60.198" size="1.778" layer="96"/>
 </instance>
 </instances>
@@
 <wire x1="215.9" y1="40.64" x2="220.98" y2="40.64" width="0.1524" layer="91"/>
 <label x="220.98" y="40.64" size="1.778" layer="95"/>
+<pinref part="J7" gate="J1" pin="SHLD"/>
+<wire x1="215.9" y1="43.18" x2="215.9" y2="40.64" width="0.1524" layer="91"/>
+<junction x="215.9" y="40.64"/>
 </segment>
 <segment>
@@
 <junction x="182.626" y="31.242"/>
 <label x="185.42" y="30.48" size="1.778" layer="95"/>
+</segment>
+<segment>
+<pinref part="GND" gate="1" pin="P"/>
+<wire x1="223.52" y1="63.5" x2="218.44" y2="63.5" width="0.1524" layer="91"/>
+<label x="218.44" y="63.5" size="1.778" layer="95"/>
 </segment>
 </net>
@@
 <label x="134.62" y="154.94" size="1.778" layer="95"/>
 <pinref part="PWR" gate="LED" pin="+"/>
-</segment>
-<segment>
-<wire x1="142.24" y1="82.55" x2="137.16" y2="82.55" width="0.1524" layer="91"/>
-<label x="133.35" y="82.55" size="1.778" layer="95"/>
-<pinref part="Q3" gate="MOS" pin="S"/>
-</segment>
-<segment>
-<wire x1="179.07" y1="81.28" x2="173.99" y2="81.28" width="0.1524" layer="91"/>
-<label x="170.18" y="81.28" size="1.778" layer="95"/>
-<pinref part="Q2" gate="MOS" pin="S"/>
 </segment>
 <segment>
@@
 <wire x1="247.015" y1="87.63" x2="237.236" y2="87.63" width="0.1524" layer="91"/>
 </segment>
-<segment>
-<wire x1="184.15" y1="86.36" x2="184.15" y2="91.44" width="0.1524" layer="91"/>
-<label x="179.705" y="92.075" size="1.778" layer="95"/>
-<pinref part="Q2" gate="MOS" pin="G"/>
-</segment>
 </net>
 <net name="D4" class="0">
@@
 <wire x1="244.475" y1="82.55" x2="237.236" y2="82.55" width="0.1524" layer="91"/>
 </segment>
-<segment>
-<wire x1="147.32" y1="87.63" x2="147.32" y2="92.71" width="0.1524" layer="91"/>
-<label x="144.78" y="91.44" size="1.778" layer="95"/>
-<pinref part="Q3" gate="MOS" pin="G"/>
-</segment>
 </net>
 <net name="D_2+" class="0">
@@
 <label x="233.68" y="55.88" size="1.778" layer="95"/>
 </segment>
-</net>
-<net name="VBET_OUT" class="0">
 <segment>
 <wire x1="10.16" y1="88.9" x2="25.4" y2="88.9" width="0.1524" layer="91"/>
@@
 <pinref part="C1" gate="C" pin="1"/>
 </segment>
+<segment>
+<pinref part="5V" gate="1" pin="P"/>
+<wire x1="218.44" y1="71.12" x2="223.52" y2="71.12" width="0.1524" layer="91"/>
+<label x="218.44" y="71.12" size="1.778" layer="95"/>
+</segment>
 </net>
 <net name="D-" class="0">
@@
 <pinref part="ASSOC" gate="LED" pin="-"/>
 <pinref part="R11" gate="R" pin="2"/>
-</segment>
-</net>
-<net name="VCC_OUT1" class="0">
-<segment>
-<wire x1="152.4" y1="82.55" x2="158.75" y2="82.55" width="0.1524" layer="91"/>
-<label x="153.67" y="82.55" size="1.778" layer="95"/>
-<pinref part="Q3" gate="MOS" pin="D"/>
-</segment>
-</net>
-<net name="VCC_OUT2" class="0">
-<segment>
-<wire x1="189.23" y1="81.28" x2="195.58" y2="81.28" width="0.1524" layer="91"/>
-<label x="190.5" y="81.28" size="1.778" layer="95"/>
-<pinref part="Q2" gate="MOS" pin="D"/>
 </segment>
 </net>
@@
 </segment>
 </net>
-<net name="N$3" class="0">
+<net name="USBC_CC1" class="0">
 <segment>
 <pinref part="J7" gate="J1" pin="CC1"/>
 <pinref part="R14" gate="R" pin="2"/>
 <wire x1="215.9" y1="48.26" x2="223.52" y2="48.26" width="0.1524" layer="91"/>
-</segment>
-</net>
-<net name="N$10" class="0">
+<label x="218.44" y="48.26" size="1.778" layer="95"/>
+</segment>
+</net>
+<net name="USBC_CC2" class="0">
 <segment>
 <pinref part="R15" gate="R" pin="2"/>
 <pinref part="J7" gate="J1" pin="CC2"/>
 <wire x1="228.6" y1="45.72" x2="215.9" y2="45.72" width="0.1524" layer="91"/>
+<label x="218.44" y="45.72" size="1.778" layer="95"/>
 </segment>
 </net>
@@
 <label x="165.1" y="35.56" size="1.778" layer="95"/>
 </segment>
+<segment>
+<pinref part="PDP" gate="1" pin="P"/>
+<wire x1="218.44" y1="66.04" x2="223.52" y2="66.04" width="0.1524" layer="91"/>
+<label x="218.44" y="66.04" size="1.778" layer="95"/>
+</segment>
 </net>
 <net name="ROOTD-" class="0">
@@
 <wire x1="154.94" y1="20.32" x2="165.1" y2="20.32" width="0.1524" layer="91"/>
 <label x="165.1" y="20.32" size="1.778" layer="95"/>
+</segment>
+<segment>
+<pinref part="PDM" gate="1" pin="P"/>
+<wire x1="223.52" y1="68.58" x2="218.44" y2="68.58" width="0.1524" layer="91"/>
+<label x="218.44" y="68.58" size="1.778" layer="95"/>
 </segment>
 </net>
@@
 </segment>
 </net>
-<net name="N$5" class="0">
+<net name="USB_OVRCUR" class="0">
 <segment>
 <pinref part="U1" gate="A" pin="~OVRCUR3"/>
@@
 <junction x="104.14" y="40.64"/>
 <junction x="104.14" y="38.1"/>
+<label x="99.06" y="35.56" size="1.778" layer="95"/>
 </segment>
 </net>
@@
 will not be understood (or retained) with this version.
 </note>
+<note version="8.3" severity="warning">
+Since Version 8.3, EAGLE supports the association of 3D packages
+with devices in libraries, schematics, and board files. Those 3D
+packages will not be understood (or retained) with this version.
+</note>
 </compatibility>

Commit message: haha yes
Parts:
- added R10: 1.5k, discrete:R-0603
- added R4, R8: 15k, discrete:R-0603
- added USB2M, USB2P, XBM, XBP: (no value), wirepad:2,15/1,0
Connections:
- net D+: now also XBP.P
- net D-: now also R4.2, XBM.P
- net D_2+: now also USB2P.P
- net D_2-: now also R8.2, USB2M.P
- net GND: now also R4.1, R8.1
- net ROOTD+: now also R10.2
- net VCC_3V3: now also R10.1
Changed lines of the file:
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@@
 <part name="PDP" library="wirepad" library_urn="urn:adsk.eagle:library:412" deviceset="2,15/1,0" device="" package3d_urn="urn:adsk.eagle:package:30831/1"/>
 <part name="GND" library="wirepad" library_urn="urn:adsk.eagle:library:412" deviceset="2,15/1,0" device="" package3d_urn="urn:adsk.eagle:package:30831/1"/>
+<part name="R4" library="discrete" library_urn="urn:adsk.eagle:library:211" deviceset="R*" device="-0603" value="15k"/>
+<part name="R8" library="discrete" library_urn="urn:adsk.eagle:library:211" deviceset="R*" device="-0603" value="15k"/>
+<part name="R10" library="discrete" library_urn="urn:adsk.eagle:library:211" deviceset="R*" device="-0603" value="1.5k"/>
+<part name="XBP" library="wirepad" library_urn="urn:adsk.eagle:library:412" deviceset="2,15/1,0" device="" package3d_urn="urn:adsk.eagle:package:30831/1"/>
+<part name="XBM" library="wirepad" library_urn="urn:adsk.eagle:library:412" deviceset="2,15/1,0" device="" package3d_urn="urn:adsk.eagle:package:30831/1"/>
+<part name="USB2P" library="wirepad" library_urn="urn:adsk.eagle:library:412" deviceset="2,15/1,0" device="" package3d_urn="urn:adsk.eagle:package:30831/1"/>
+<part name="USB2M" library="wirepad" library_urn="urn:adsk.eagle:library:412" deviceset="2,15/1,0" device="" package3d_urn="urn:adsk.eagle:package:30831/1"/>
 </parts>
 <sheets>
@@
 <attribute name="NAME" x="207.137" y="62.8142" size="1.778" layer="95"/>
 <attribute name="VALUE" x="214.757" y="60.198" size="1.778" layer="96"/>
+</instance>
+<instance part="R4" gate="R" x="176.276" y="18.542" smashed="yes" rot="R180">
+<attribute name="NAME" x="178.816" y="21.082" size="1.778" layer="95" ratio="10" rot="R180"/>
+<attribute name="VALUE" x="178.181" y="17.272" size="1.778" layer="96" ratio="10" rot="R180"/>
+</instance>
+<instance part="R8" gate="R" x="176.276" y="16.002" smashed="yes" rot="R180">
+<attribute name="NAME" x="178.816" y="18.542" size="1.778" layer="95" ratio="10" rot="R180"/>
+<attribute name="VALUE" x="178.181" y="14.732" size="1.778" layer="96" ratio="10" rot="R180"/>
+</instance>
+<instance part="R10" gate="R" x="161.036" y="41.402" smashed="yes" rot="R270">
+<attribute name="NAME" x="158.496" y="43.942" size="1.778" layer="95" ratio="10" rot="R270"/>
+<attribute name="VALUE" x="162.306" y="43.307" size="1.778" layer="96" ratio="10" rot="R270"/>
+</instance>
+<instance part="XBP" gate="1" x="205.74" y="78.74" smashed="yes">
+<attribute name="NAME" x="196.977" y="78.0542" size="1.778" layer="95"/>
+<attribute name="VALUE" x="204.597" y="75.438" size="1.778" layer="96"/>
+</instance>
+<instance part="XBM" gate="1" x="205.74" y="76.2" smashed="yes">
+<attribute name="NAME" x="196.977" y="75.5142" size="1.778" layer="95"/>
+<attribute name="VALUE" x="204.597" y="72.898" size="1.778" layer="96"/>
+</instance>
+<instance part="USB2P" gate="1" x="205.74" y="83.82" smashed="yes">
+<attribute name="NAME" x="196.977" y="83.1342" size="1.778" layer="95"/>
+<attribute name="VALUE" x="204.597" y="80.518" size="1.778" layer="96"/>
+</instance>
+<instance part="USB2M" gate="1" x="205.74" y="81.28" smashed="yes">
+<attribute name="NAME" x="196.977" y="80.5942" size="1.778" layer="95"/>
+<attribute name="VALUE" x="204.597" y="77.978" size="1.778" layer="96"/>
 </instance>
 </instances>
@@
 <junction x="182.626" y="31.242"/>
 <label x="185.42" y="30.48" size="1.778" layer="95"/>
+<pinref part="R4" gate="R" pin="1"/>
+<wire x1="180.086" y1="18.542" x2="182.626" y2="18.542" width="0.1524" layer="91"/>
+<wire x1="182.626" y1="18.542" x2="182.626" y2="31.242" width="0.1524" layer="91"/>
+<pinref part="R8" gate="R" pin="1"/>
+<wire x1="180.086" y1="16.002" x2="182.626" y2="16.002" width="0.1524" layer="91"/>
+<wire x1="182.626" y1="16.002" x2="182.626" y2="31.242" width="0.1524" layer="91"/>
 </segment>
 <segment>
@@
 <wire x1="91.186" y1="27.94" x2="91.44" y2="27.94" width="0.1524" layer="91"/>
 </segment>
+<segment>
+<pinref part="R10" gate="R" pin="1"/>
+<wire x1="161.036" y1="45.212" x2="161.036" y2="48.26" width="0.1524" layer="91"/>
+<label x="162.56" y="45.72" size="1.778" layer="95"/>
+</segment>
 </net>
 <net name="D6" class="0">
@@
 <segment>
 <pinref part="U1" gate="A" pin="DM2"/>
-<wire x1="154.94" y1="15.24" x2="165.1" y2="15.24" width="0.1524" layer="91"/>
+<wire x1="154.94" y1="15.24" x2="172.466" y2="15.24" width="0.1524" layer="91"/>
 <label x="165.1" y="15.24" size="1.778" layer="95"/>
+<pinref part="R8" gate="R" pin="2"/>
+<wire x1="172.466" y1="16.002" x2="172.466" y2="15.24" width="0.1524" layer="91"/>
+</segment>
+<segment>
+<pinref part="USB2M" gate="1" pin="P"/>
+<wire x1="208.28" y1="81.28" x2="210.82" y2="81.28" width="0.1524" layer="91"/>
+<label x="210.82" y="81.28" size="1.778" layer="95"/>
 </segment>
 </net>
@@
 <pinref part="R13" gate="R" pin="2"/>
 <wire x1="175.006" y1="31.242" x2="175.006" y2="30.48" width="0.1524" layer="91"/>
+</segment>
+<segment>
+<pinref part="USB2P" gate="1" pin="P"/>
+<wire x1="210.82" y1="83.82" x2="208.28" y2="83.82" width="0.1524" layer="91"/>
+<label x="210.82" y="83.82" size="1.778" layer="95"/>
 </segment>
 </net>
@@
 <segment>
 <pinref part="U1" gate="A" pin="DM1"/>
-<wire x1="154.94" y1="17.78" x2="165.1" y2="17.78" width="0.1524" layer="91"/>
+<wire x1="154.94" y1="17.78" x2="172.466" y2="17.78" width="0.1524" layer="91"/>
 <label x="165.1" y="17.78" size="1.778" layer="95"/>
+<pinref part="R4" gate="R" pin="2"/>
+<wire x1="172.466" y1="17.78" x2="172.466" y2="18.542" width="0.1524" layer="91"/>
+</segment>
+<segment>
+<pinref part="XBM" gate="1" pin="P"/>
+<wire x1="210.82" y1="76.2" x2="208.28" y2="76.2" width="0.1524" layer="91"/>
+<label x="210.82" y="76.2" size="1.778" layer="95"/>
 </segment>
 </net>
@@
 <pinref part="R12" gate="R" pin="2"/>
 <wire x1="175.006" y1="33.782" x2="175.006" y2="33.02" width="0.1524" layer="91"/>
+</segment>
+<segment>
+<pinref part="XBP" gate="1" pin="P"/>
+<wire x1="208.28" y1="78.74" x2="210.82" y2="78.74" width="0.1524" layer="91"/>
+<label x="210.82" y="78.74" size="1.778" layer="95"/>
 </segment>
 </net>
@@
 <segment>
 <pinref part="U1" gate="A" pin="DP0"/>
-<wire x1="154.94" y1="35.56" x2="165.1" y2="35.56" width="0.1524" layer="91"/>
+<wire x1="154.94" y1="35.56" x2="161.036" y2="35.56" width="0.1524" layer="91"/>
 <label x="165.1" y="35.56" size="1.778" layer="95"/>
-</segment>
-<segment>
+<pinref part="R10" gate="R" pin="2"/>
+<wire x1="162.56" y1="35.56" x2="165.1" y2="35.56" width="0.1524" layer="91"/>
+<wire x1="161.036" y1="37.592" x2="161.036" y2="35.56" width="0.1524" layer="91"/>
+<wire x1="161.036" y1="35.56" x2="162.56" y2="35.56" width="0.1524" layer="91"/>
+</segment>
+<segment>

Commit message: plz dont break
Other:
- note removed: "RC for usb hub reset"
- moved on the sheet: C3, C6, R1, R2, R3, R7, R9, RX, TX, U4
